File: sensordio.brd (EAGLE design)
At the start: 100 x 80 mm, 16 parts, among them IC1 PCA9534D, IC2 ULN2003AD

Commit message: Whoops, missing from previous.
Parts:
- moved U$1 71.7 mm to (21.6, 22.9)
- moved C2 19.2 mm to (6.35, 2.54), turned to 270 degrees
- moved C3 19.1 mm to (12.7, 2.54), turned to 270 degrees
- moved C1 19.1 mm to (19.1, 2.54), turned to 270 degrees
- moved JIO2 5.24 mm to (50.8, 12.7), turned to 90 degrees
- moved IC2 4.02 mm to (43.2, 12.7), turned to 270 degrees
- moved R1 3.59 mm to (16.5, 20.3), turned to 270 degrees
- moved R12 2.54 mm to (7.62, 20.3), turned to 270 degrees
- moved R11 1.80 mm to (11.4, 20.3), turned to 270 degrees
- turned JIO1 to 90 degrees
Other:
- board size 100 x 80 mm -> 54.3 x 25.4 mm
